File: hardware/Standard_18650/18650.sch (KiCad schematic (older format))
At the start: 56 parts, among them J2 Battery, J3 GPIO, J4 USB_B_Micro, J5 Power, J6 LEDs, J7 GPIO, Q1 BSS806N, Q2 BSS806N, Q3 BSS806N, Q4 BSS806N, SW1 Mode, SW2 Power, U1 STM32F411CE, U2 AP2210N-3.3TRG1, U3 BQ21040, U4 ESD7002WTT1G, Y1 24Mhz

Commit message: buck boost IC
Added the TPS63806 symbol to the local library. Replaced the linear regulator that powers the 3.3V rail in Standard_18650 with the buck boost IC TPS63806.
Parts:
- removed U2: AP2210N-3.3TRG1, Package_TO_SOT_SMD:SOT-23, symbol Jeremy:AP2210-3.3TRG1
- added R? (x2): 10K, symbol Device:R_Small
- added R?: 511K, symbol Device:R_Small
- added R?: 91K, symbol Device:R_Small
- added U?: TPS63806, symbol Standard_18650:TPS63806
- U3: symbol Jeremy:BQ21040 -> 18650-rescue:BQ21040-Jeremy
- U4: symbol Jeremy:ESD7002WTT1G -> 18650-rescue:ESD7002WTT1G-Jeremy
Connections:
- wire segments 227 -> 249
Changed lines of the file:
@@
 EESchema Schematic File Version 4
-EELAYER 30 0
+LIBS:18650-cache
+EELAYER 29 0
 EELAYER END
 $Descr A4 11693 8268
@@
 	0    1    1    0
 $EndComp
-$Comp
-L Jeremy:AP2210-3.3TRG1 U2
-U 1 1 5CD3E552
-P 5650 6950
-F 0 "U2" H 5750 6650 50  0000 C CNN
-F 1 "AP2210N-3.3TRG1" H 5925 7134 50  0000 C CNN
-F 2 "Package_TO_SOT_SMD:SOT-23" H 5600 7350 50  0001 C CNN
-F 3 "" H 5600 7350 50  0001 C CNN
-F 4 "AP2210N-3.3TRG1" H 5650 6950 50  0001 C CNN "MPN"
-	1    5650 6950
-	1    0    0    -1
-$EndComp
-Text Notes 5000 6500 0    50   ~ 0
+Text Notes 4450 5000 0    50   ~ 0
 3.3v Power
-Text Label 5200 6900 2    50   ~ 0
+Text Label 4750 5700 2    50   ~ 0
 VIN
 $Comp
 L power:GND #PWR0108
 U 1 1 5BD85B6B
-P 5900 7500
-F 0 "#PWR0108" H 5900 7250 50  0001 C CNN
-F 1 "GND" H 5905 7327 50  0000 C CNN
-F 2 "" H 5900 7500 50  0001 C CNN
-F 3 "" H 5900 7500 50  0001 C CNN
-	1    5900 7500
+P 5500 6650
+F 0 "#PWR0108" H 5500 6400 50  0001 C CNN
+F 1 "GND" H 5505 6477 50  0000 C CNN
+F 2 "" H 5500 6650 50  0001 C CNN
+F 3 "" H 5500 6650 50  0001 C CNN
+	1    5500 6650
 	1    0    0    -1
 $EndComp
@@
 L power:+3V3 #PWR0102
 U 1 1 5BD53A46
-P 6650 6800
-F 0 "#PWR0102" H 6650 6650 50  0001 C CNN
-F 1 "+3V3" H 6665 6973 50  0000 C CNN
-F 2 "" H 6650 6800 50  0001 C CNN
-F 3 "" H 6650 6800 50  0001 C CNN
-	1    6650 6800
+P 6900 5600
+F 0 "#PWR0102" H 6900 5450 50  0001 C CNN
+F 1 "+3V3" H 6915 5773 50  0000 C CNN
+F 2 "" H 6900 5600 50  0001 C CNN
+F 3 "" H 6900 5600 50  0001 C CNN
+	1    6900 5600
 	1    0    0    -1
 $EndComp
@@
 $EndComp
 Wire Wire Line
-	5200 6900 5350 6900
+	4750 5700 4900 5700
 $Comp
 L Device:C C6
 U 1 1 5DA6D345
-P 5350 7100
-F 0 "C6" H 5400 7000 50  0000 L CNN
-F 1 "1uF" H 5400 7200 50  0000 L CNN
-F 2 "Capacitor_SMD:C_0603_1608Metric" H 5388 6950 50  0001 C CNN
-F 3 "~" H 5350 7100 50  0001 C CNN
-F 4 "0603" H 5350 7100 50  0001 C CNN "Package"
-	1    5350 7100
-	1    0    0    -1
-$EndComp
-Wire Wire Line
-	5350 6950 5350 6900
-Connection ~ 5350 6900
-Wire Wire Line
-	5350 6900 5500 6900
-Wire Wire Line
-	5350 7250 5350 7350
-Wire Wire Line
-	5350 7350 5900 7350
-Wire Wire Line
-	5900 7350 5900 7500
-Connection ~ 5900 7350
-Wire Wire Line
-	6350 6900 6450 6900
-Wire Wire Line
-	6650 6900 6650 6800
-Wire Wire Line
-	6450 6950 6450 6900
-Connection ~ 6450 6900
-Wire Wire Line
-	6450 6900 6650 6900
+P 4900 5900
+F 0 "C6" H 4950 5800 50  0000 L CNN
+F 1 "1uF" H 4950 6000 50  0000 L CNN
+F 2 "Capacitor_SMD:C_0603_1608Metric" H 4938 5750 50  0001 C CNN
+F 3 "~" H 4900 5900 50  0001 C CNN
+F 4 "0603" H 4900 5900 50  0001 C CNN "Package"
+	1    4900 5900
+	1    0    0    -1
+$EndComp
+Wire Wire Line
+	4900 5750 4900 5700
+Connection ~ 4900 5700
+Wire Wire Line
+	6900 5700 6900 5600
+Wire Wire Line
+	6900 5750 6900 5700
 $Comp
 L Device:C C12
 U 1 1 5DAD6F5D
-P 6450 7100
-F 0 "C12" H 6550 7000 50  0000 L CNN
-F 1 "2.2uF" H 6550 7200 50  0000 L CNN
-F 2 "Capacitor_SMD:C_0603_1608Metric" H 6488 6950 50  0001 C CNN
-F 3 "" H 6450 7100 50  0001 C CNN
-F 4 "0603" H 6450 7100 50  0001 C CNN "Package"
-F 5 "CL10A225KO8NNNC" H 6450 7100 50  0001 C CNN "MPN"
-	1    6450 7100
-	1    0    0    -1
-$EndComp
-Wire Wire Line
-	6450 7250 6450 7350
-Wire Wire Line
-	6450 7350 5900 7350
-Wire Notes Line
-	5000 6500 5000 7750
+P 6900 5900
+F 0 "C12" H 7000 5800 50  0000 L CNN
+F 1 "2.2uF" H 7000 6000 50  0000 L CNN
+F 2 "Capacitor_SMD:C_0603_1608Metric" H 6938 5750 50  0001 C CNN
+F 3 "" H 6900 5900 50  0001 C CNN
+F 4 "0603" H 6900 5900 50  0001 C CNN "Package"
+F 5 "CL10A225KO8NNNC" H 6900 5900 50  0001 C CNN "MPN"
+	1    6900 5900
+	1    0    0    -1
+$EndComp
+Wire Notes Line
+	4450 5000 4450 6250
 Wire Notes Line
 	6850 6500 6850 7750
 Wire Notes Line
-	5000 6500 6850 6500
+	4450 5000 6300 5000
 Wire Notes Line
 	5000 7750 6850 7750
@@
 	3100 6950 3800 6950
 $Comp
-L Jeremy:ESD7002WTT1G U4
+L 18650-rescue:ESD7002WTT1G-Jeremy U4
 U 1 1 5DA9EA0D
 P 4200 7300
@@
 	1400 3300 1650 3300
 $Comp
-L Jeremy:BQ21040 U3
+L 18650-rescue:BQ21040-Jeremy U3
 U 1 1 5DB9B819
 P 8900 5050
@@
 Connection ~ 2650 5750
 NoConn ~ 3100 7050
+Wire Wire Line
+	4900 5700 5150 5700
+Wire Wire Line
+	5450 5800 5450 5700
+Wire Wire Line
+	4900 6350 5150 6350
+Wire Wire Line
+	4900 6050 4900 6350
+Wire Wire Line
+	5500 6350 5500 6650
+Connection ~ 5500 6350
+Wire Wire Line
+	6350 5800 6350 5700
+$Comp
+L Device:R_Small R?
+U 1 1 5ECBDE24
+P 5150 5900
+F 0 "R?" H 5209 5946 50  0000 L CNN
+F 1 "10K" H 5209 5855 50  0000 L CNN
+F 2 "" H 5150 5900 50  0001 C CNN
+F 3 "~" H 5150 5900 50  0001 C CNN
+	1    5150 5900
+	1    0    0    -1
+$EndComp
+$Comp
+L Standard_18650:TPS63806 U?
+U 1 1 5ECD1700
+P 5900 5850
+F 0 "U?" H 5900 5261 50  0000 C CNN
+F 1 "TPS63806" H 5900 5170 50  0000 C CNN
+F 2 "" H 6250 6450 50  0001 C CNN
+F 3 "" H 6250 6450 50  0001 C CNN
+	1    5900 5850
+	1    0    0    -1
+$EndComp
+Wire Wire Line
+	5500 6350 5700 6350
+Connection ~ 5450 5700
+Connection ~ 6350 5700
+Wire Wire Line
+	5700 6350 5800 6350
+Connection ~ 5700 6350
+Connection ~ 5800 6350
+Wire Wire Line
+	5800 6350 6050 6350
+Wire Wire Line
+	5450 5900 5350 5900
+Wire Wire Line
+	5350 5900 5350 6000
+Wire Wire Line
+	5350 6000 5150 6000
+Wire Wire Line
+	5150 5800 5150 5700
+Connection ~ 5150 5700
+Wire Wire Line
+	5150 5700 5450 5700
+$Comp
+L Device:R_Small R?
+U 1 1 5ED348A1
+P 5150 6150
+F 0 "R?" H 5209 6196 50  0000 L CNN
+F 1 "10K" H 5209 6105 50  0000 L CNN
+F 2 "" H 5150 6150 50  0001 C CNN
+F 3 "~" H 5150 6150 50  0001 C CNN
+	1    5150 6150
+	1    0    0    -1
+$EndComp
+Wire Wire Line
+	5150 6050 5150 6000
+Connection ~ 5150 6000
+Wire Wire Line
+	5150 6250 5150 6350
+Connection ~ 5150 6350
+Wire Wire Line
+	5150 6350 5500 6350
+$Comp
+L Device:R_Small R?
+U 1 1 5ED58939
+P 6550 5850
+F 0 "R?" H 6609 5896 50  0000 L CNN
+F 1 "511K" H 6609 5805 50  0000 L CNN
+F 2 "" H 6550 5850 50  0001 C CNN
+F 3 "~" H 6550 5850 50  0001 C CNN
+	1    6550 5850
+	1    0    0    -1
+$EndComp
+$Comp
+L Device:R_Small R?
+U 1 1 5ED5A245
+P 6550 6250
+F 0 "R?" H 6609 6296 50  0000 L CNN
+F 1 "91K" H 6609 6205 50  0000 L CNN
+F 2 "" H 6550 6250 50  0001 C CNN
+F 3 "~" H 6550 6250 50  0001 C CNN
+	1    6550 6250
+	1    0    0    -1
+$EndComp
+Connection ~ 6900 5700
+Wire Wire Line
+	6350 5700 6550 5700
+Wire Wire Line
+	6550 6000 6550 5950
+Wire Wire Line
+	6550 5750 6550 5700
+Connection ~ 6550 5700
+Wire Wire Line
+	6550 5700 6900 5700
+Wire Wire Line
+	6350 6000 6550 6000
+Wire Wire Line
+	6550 6150 6550 6000
+Connection ~ 6550 6000
+Wire Wire Line
+	6550 6350 6050 6350
+Connection ~ 6050 6350
+Wire Wire Line
+	6550 6350 6900 6350
+Wire Wire Line
+	6900 6050 6900 6350
+Connection ~ 6550 6350
+Wire Wire Line
+	5800 5350 5700 5350
+Wire Wire Line
+	6000 5350 6100 5350
+Wire Wire Line
+	5700 5350 5000 5350
+Connection ~ 5700 5350
+Wire Wire Line
+	6100 5350 6600 5350
+Connection ~ 6100 5350
 $EndSCHEMATC
